File: TSAL/untitled.kicad_sch (KiCad schematic)
At the start: 29 parts, among them J3 TE 770966-2, J4 TE 770966-2, Q4 STD7NK40Z, T1 11328-T078, U6 LT8316IFE#PBF

Commit message: resisitor change
Parts:
- C7: value 0.1u -> 100nF
Changed lines of the file:
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@@
       (effects (font (size 1.27 1.27)) (justify left))
     )
-    (property "Value" "0.1u" (id 1) (at 62.23 100.33 0)
+    (property "Value" "100nF" (id 1) (at 62.23 100.33 0)
       (effects (font (size 1.27 1.27)) (justify left))
     )
