File: TSAL/PCB.kicad_sch (KiCad schematic)
At the start: 38 parts, among them J1 TE 770966-2, J2 JST B04B-XASK, Q1 IRLZ44N, Q2 2N3904, Q3 IRLZ44N, U1 TL431D, U2 LMV331, U3 VRB1205YMD-6WR3, U4 NSL-32, U5 LM555xN

Commit message: Changed opto-isolator
Parts:
- removed Q2: 2N3904, Package_TO_SOT_THT:TO-92_Inline, symbol Transistor_BJT:2N3904
- removed U4: NSL-32, OptoDevice:Luna_NSL-32, symbol Isolator:NSL-32
- added Q2: MMBT3904, Package_TO_SOT_SMD:SOT-23, symbol Transistor_BJT:MMBT3904
- added U4: LTV-817S, Package_DIP:SMDIP-4_W9.53mm, symbol Isolator:LTV-817S
- C1: footprint Potentiometer_SMD:Potentiometer_Bourns_3314J_Vertical -> Capacitor_SMD:CP_Elec_6.3x7.7
- Q1, Q3: footprint Package_TO_SOT_THT:TO-220-3_Vertical -> Package_TO_SOT_SMD:TO-263-2
- U5: footprint Package_DIP:DIP-8_W7.62mm -> Package_SO:SOIC-8_3.9x4.9mm_P1.27mm
Connections:
- net +12V: now also U4.4; no longer C5.1
- net +5V: now also C5.1
- net GND: now also Q2.2 (E)
- net at R16.1, R7.1, R8.1: now also U4.3
- net at R16.2: now also Q2.1 (B)
- net at R6.2: now also U4.1
- net at U2.4: now also U4.2
- net at R9.1, U5.4 (R): now also Q2.3 (C)
Changed lines of the file:
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@@
       (effects (font (size 1.27 1.27)) (justify left))
     )
-    (property "Footprint" "Package_TO_SOT_THT:TO-220-3_Vertical" (id 2) (at 246.38 108.585 0)
+    (property "Footprint" "Package_TO_SOT_SMD:TO-263-2" (id 2) (at 246.38 108.585 0)
       (effects (font (size 1.27 1.27) italic) (justify left) hide)
     )
@@
     (pin "2")
   )
+  (symbol (lib_id "Isolator:LTV-817S") (at 113.03 120.65 0) (unit 1)
+    (in_bom yes) (on_board yes) (fields_autoplaced)
+    (property "Reference" "U4" (id 0) (at 113.03 111.76 0))
+    (property "Value" "LTV-817S" (id 1) (at 113.03 114.3 0))
+    (property "Footprint" "Package_DIP:SMDIP-4_W9.53mm" (id 2) (at 113.03 128.27 0)
+      (effects (font (size 1.27 1.27)) hide)
+    )
+    (property "Datasheet" "http://www.us.liteon.com/downloads/LTV-817-827-847.PDF" (id 3) (at 104.14 113.03 0)
+      (effects (font (size 1.27 1.27)) hide)
+    )
+    (pin "1")
+    (pin "2")
+    (pin "3")
+    (pin "4")
+  )
   (symbol (lib_id "Device:D_TVS") (at 127 64.77 90) (unit 1)
     (in_bom yes) (on_board yes)
@@
     (pin "2")
   )
+  (symbol (lib_id "Transistor_BJT:MMBT3904") (at 140.97 123.19 0) (unit 1)
+    (in_bom yes) (on_board yes) (fields_autoplaced)
+    (property "Reference" "Q2" (id 0) (at 146.05 121.9199 0)
+      (effects (font (size 1.27 1.27)) (justify left))
+    )
+    (property "Value" "MMBT3904" (id 1) (at 146.05 124.4599 0)
+      (effects (font (size 1.27 1.27)) (justify left))
+    )
+    (property "Footprint" "Package_TO_SOT_SMD:SOT-23" (id 2) (at 146.05 125.095 0)
+      (effects (font (size 1.27 1.27) italic) (justify left) hide)
+    )
+    (property "Datasheet" "https://www.onsemi.com/pub/Collateral/2N3903-D.PDF" (id 3) (at 140.97 123.19 0)
+      (effects (font (size 1.27 1.27)) (justify left) hide)
+    )
+    (pin "1")
+    (pin "2")
+    (pin "3")
+  )
   (symbol (lib_id "power:GND") (at 196.85 130.81 0) (unit 1)
     (in_bom yes) (on_board yes) (fields_autoplaced)
@@
       (effects (font (size 1.27 1.27)) (justify left))
     )
-    (property "Footprint" "Package_TO_SOT_THT:TO-220-3_Vertical" (id 2) (at 144.78 167.005 0)
+    (property "Footprint" "Package_TO_SOT_SMD:TO-263-2" (id 2) (at 144.78 167.005 0)
       (effects (font (size 1.27 1.27) italic) (justify left) hide)
     )
@@
       (effects (font (size 1.27 1.27)) (justify left))
     )
-    (property "Footprint" "Potentiometer_SMD:Potentiometer_Bourns_3314J_Vertical" (id 2) (at 95.5548 68.58 0)
+    (property "Footprint" "Capacitor_SMD:CP_Elec_6.3x7.7" (id 2) (at 95.5548 68.58 0)
       (effects (font (size 1.27 1.27)) hide)
     )
@@
     (pin "1")
     (pin "2")
-  )
-  (symbol (lib_id "power:+12V") (at 80.01 106.68 0) (unit 1)
-    (in_bom yes) (on_board yes) (fields_autoplaced)
-    (property "Reference" "#PWR0101" (id 0) (at 80.01 110.49 0)
-      (effects (font (size 1.27 1.27)) hide)
-    )
-    (property "Value" "+12V" (id 1) (at 80.01 101.6 0))
-    (property "Footprint" "" (id 2) (at 80.01 106.68 0)
-      (effects (font (size 1.27 1.27)) hide)
-    )
-    (property "Datasheet" "" (id 3) (at 80.01 106.68 0)
-      (effects (font (size 1.27 1.27)) hide)
-    )
-    (pin "1")
   )
   (symbol (lib_id "Device:R") (at 123.19 171.45 0) (unit 1)
@@
     )
     (property "Datasheet" "" (id 3) (at 82.55 115.57 0)
+      (effects (font (size 1.27 1.27)) hide)
+    )
+    (pin "1")
+  )
+  (symbol (lib_id "power:+5V") (at 80.01 106.68 0) (unit 1)
+    (in_bom yes) (on_board yes) (fields_autoplaced)
+    (property "Reference" "#PWR0101" (id 0) (at 80.01 110.49 0)
+      (effects (font (size 1.27 1.27)) hide)
+    )
+    (property "Value" "+5V" (id 1) (at 80.01 101.6 0))
+    (property "Footprint" "" (id 2) (at 80.01 106.68 0)
+      (effects (font (size 1.27 1.27)) hide)
+    )
+    (property "Datasheet" "" (id 3) (at 80.01 106.68 0)
       (effects (font (size 1.27 1.27)) hide)
     )
@@
       (effects (font (size 1.27 1.27)) (justify left))
     )
-    (property "Footprint" "Package_DIP:DIP-8_W7.62mm" (id 2) (at 213.36 121.92 0)
+    (property "Footprint" "Package_SO:SOIC-8_3.9x4.9mm_P1.27mm" (id 2) (at 213.36 121.92 0)
       (effects (font (size 1.27 1.27)) hide)
     )
@@
     (pin "1")
     (pin "2")
-  )
-  (symbol (lib_id "Isolator:NSL-32") (at 113.03 120.65 0) (unit 1)
-    (in_bom yes) (on_board yes) (fields_autoplaced)
-    (property "Reference" "U4" (id 0) (at 113.03 111.76 0))
-    (property "Value" "NSL-32" (id 1) (at 113.03 114.3 0))
-    (property "Footprint" "OptoDevice:Luna_NSL-32" (id 2) (at 113.03 128.27 0)
-      (effects (font (size 1.27 1.27)) hide)
-    )
-    (property "Datasheet" "http://lunainc.com/wp-content/uploads/2016/06/NSL-32.pdf" (id 3) (at 114.3 120.65 0)
-      (effects (font (size 1.27 1.27)) hide)
-    )
-    (pin "1")
-    (pin "2")
-    (pin "3")
-    (pin "4")
   )
   (symbol (lib_id "Reference_Voltage:TL431D") (at 49.53 82.55 90) (unit 1)
@@
     (pin "1")
   )
-  (symbol (lib_id "Transistor_BJT:2N3904") (at 140.97 123.19 0) (unit 1)
-    (in_bom yes) (on_board yes) (fields_autoplaced)
-    (property "Reference" "Q2" (id 0) (at 146.05 121.9199 0)
-      (effects (font (size 1.27 1.27)) (justify left))
-    )
-    (property "Value" "2N3904" (id 1) (at 146.05 124.4599 0)
-      (effects (font (size 1.27 1.27)) (justify left))
-    )
-    (property "Footprint" "Package_TO_SOT_THT:TO-92_Inline" (id 2) (at 146.05 125.095 0)
-      (effects (font (size 1.27 1.27) italic) (justify left) hide)
-    )
-    (property "Datasheet" "https://www.onsemi.com/pub/Collateral/2N3903-D.PDF" (id 3) (at 140.97 123.19 0)
-      (effects (font (size 1.27 1.27)) (justify left) hide)
-    )
-    (pin "1")
-    (pin "2")
-    (pin "3")
-  )
   (symbol (lib_id "Device:R") (at 152.4 139.7 180) (unit 1)
     (in_bom yes) (on_board yes) (fields_autoplaced)
@@
       (reference "#PWR026") (unit 1) (value "+12V") (footprint "")
     )
-    (path "/865ae473-710e-44cb-8359-e5a8b3ee3a14"
-      (reference "#PWR0101") (unit 1) (value "+12V") (footprint "")
+    (path "/97a0b257-9ae9-471d-af82-d155cf4367e4"
+      (reference "#PWR0101") (unit 1) (value "+5V") (footprint "")
     )
     (path "/2ec14064-10a7-48ca-a71c-14c96f5ad6c0"
@@
     )
     (path "/83cea282-d52e-4e73-bdb5-72e95f42417a"
-      (reference "C1") (unit 1) (value "100u") (footprint "Potentiometer_SMD:Potentiometer_Bourns_3314J_Vertical")
+      (reference "C1") (unit 1) (value "100u") (footprint "Capacitor_SMD:CP_Elec_6.3x7.7")
     )
     (path "/429dad24-8590-49ac-a832-ab6435021168"
@@
     )
     (path "/7dfcbc7d-a633-44d1-8c93-de089712d310"
-      (reference "Q1") (unit 1) (value "IRLZ44N") (footprint "Package_TO_SOT_THT:TO-220-3_Vertical")
-    )
-    (path "/f42ffa4b-490a-4a75-8cf2-84758377a22a"
-      (reference "Q2") (unit 1) (value "2N3904") (footprint "Package_TO_SOT_THT:TO-92_Inline")
+      (reference "Q1") (unit 1) (value "IRLZ44N") (footprint "Package_TO_SOT_SMD:TO-263-2")
+    )
+    (path "/78f94064-a31d-4dcd-9046-06909c0e11ba"
+      (reference "Q2") (unit 1) (value "MMBT3904") (footprint "Package_TO_SOT_SMD:SOT-23")
     )
     (path "/203c24c0-a839-4c99-818e-dbf4875c3368"
-      (reference "Q3") (unit 1) (value "IRLZ44N") (footprint "Package_TO_SOT_THT:TO-220-3_Vertical")
+      (reference "Q3") (unit 1) (value "IRLZ44N") (footprint "Package_TO_SOT_SMD:TO-263-2")
     )
     (path "/f2108bfb-38ea-4e94-955c-eefc1ef519d2/4d000382-04b6-4720-bc4d-f38198b55000"
@@
       (reference "U3") (unit 1) (value "VRB1205YMD-6WR3") (footprint "VRB1205YMD-6WR3:VRB1205YMD-6WR3")
     )
-    (path "/e2c3a487-691b-46d7-898b-af3bd5be3fde"
-      (reference "U4") (unit 1) (value "NSL-32") (footprint "OptoDevice:Luna_NSL-32")
+    (path "/706fc87c-07e2-4407-ab34-66036b9da5a8"
+      (reference "U4") (unit 1) (value "LTV-817S") (footprint "Package_DIP:SMDIP-4_W9.53mm")
     )
     (path "/cf57b224-3a34-4dfe-953b-364e08471a95"
-      (reference "U5") (unit 1) (value "LM555xN") (footprint "Package_DIP:DIP-8_W7.62mm")
+      (reference "U5") (unit 1) (value "LM555xN") (footprint "Package_SO:SOIC-8_3.9x4.9mm_P1.27mm")
     )
     (path "/f2108bfb-38ea-4e94-955c-eefc1ef519d2/f84fad3d-971e-4ee7-9445-38f9e3b0b34f"

Commit message: resisitor change
Parts:
- added R28, R29: 500k, Resistor_SMD:R_1206_3216Metric, symbol Device:R
- C4: value 1microF -> 1u
- R3, R4: value 1M -> 500k
Connections:
- net at D1.1 (K), R5.1, U2.3 (-): now also R29.2; no longer R4.2
- new net: R28.1, R4.2
- new net: R28.2, R29.1
Changed lines of the file:
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@@
     (company "Bronco Racing")
   )
+  (junction (at 49.53 129.54) (diameter 0) (color 0 0 0 0)
+  )
   (junction (at 210.82 116.84) (diameter 0) (color 0 0 0 0)
   )
@@
   (junction (at 96.52 68.58) (diameter 0) (color 0 0 0 0)
   )
-  (junction (at 49.53 129.54) (diameter 0) (color 0 0 0 0)
-  )
   (wire (pts (xy 210.82 124.46) (xy 181.61 124.46))
     (stroke (width 0) (type default) (color 0 0 0 0))
@@
     (stroke (width 0) (type default) (color 0 0 0 0))
   )
+  (wire (pts (xy 40.64 129.54) (xy 40.64 127))
+    (stroke (width 0) (type default) (color 0 0 0 0))
+  )
   (wire (pts (xy 256.54 118.11) (xy 256.54 101.6))
     (stroke (width 0) (type default) (color 0 0 0 0))
@@
     (stroke (width 0) (type default) (color 0 0 0 0))
   )
-  (wire (pts (xy 49.53 105.41) (xy 49.53 109.22))
-    (stroke (width 0) (type default) (color 0 0 0 0))
-  )
   (wire (pts (xy 250.19 147.32) (xy 232.41 147.32))
     (stroke (width 0) (type default) (color 0 0 0 0))
@@
     (stroke (width 0) (type default) (color 0 0 0 0))
   )
-  (wire (pts (xy 49.53 116.84) (xy 49.53 118.11))
-    (stroke (width 0) (type default) (color 0 0 0 0))
-  )
   (wire (pts (xy 143.51 115.57) (xy 143.51 116.84))
     (stroke (width 0) (type default) (color 0 0 0 0))
@@
     (stroke (width 0) (type default) (color 0 0 0 0))
   )
+  (wire (pts (xy 41.91 129.54) (xy 40.64 129.54))
+    (stroke (width 0) (type default) (color 0 0 0 0))
+  )
   (wire (pts (xy 236.22 144.78) (xy 242.57 144.78))
     (stroke (width 0) (type default) (color 0 0 0 0))
@@
   )
   (wire (pts (xy 248.92 152.4) (xy 250.19 152.4))
-    (stroke (width 0) (type default) (color 0 0 0 0))
-  )
-  (wire (pts (xy 49.53 125.73) (xy 49.53 129.54))
     (stroke (width 0) (type default) (color 0 0 0 0))
   )
@@
     (pin "2")
   )
-  (symbol (lib_id "power_symbols:TS+") (at 49.53 105.41 0) (unit 1)
-    (in_bom yes) (on_board yes) (fields_autoplaced)
-    (property "Reference" "#PWR05" (id 0) (at 49.53 109.22 0)
-      (effects (font (size 1.27 1.27)) hide)
-    )
-    (property "Value" "TS+" (id 1) (at 49.53 100.33 0))
-    (property "Footprint" "" (id 2) (at 49.53 105.41 0)
-      (effects (font (size 1.27 1.27)) hide)
-    )
-    (property "Datasheet" "" (id 3) (at 49.53 105.41 0)
+  (symbol (lib_id "power_symbols:TS+") (at 40.64 104.14 0) (unit 1)
+    (in_bom yes) (on_board yes) (fields_autoplaced)
+    (property "Reference" "#PWR05" (id 0) (at 40.64 107.95 0)
+      (effects (font (size 1.27 1.27)) hide)
+    )
+    (property "Value" "TS+" (id 1) (at 40.64 99.06 0))
+    (property "Footprint" "" (id 2) (at 40.64 104.14 0)
+      (effects (font (size 1.27 1.27)) hide)
+    )
+    (property "Datasheet" "" (id 3) (at 40.64 104.14 0)
       (effects (font (size 1.27 1.27)) hide)
     )
@@
       (effects (font (size 1.27 1.27)) (justify left))
     )
-    (property "Value" "1microF" (id 1) (at 220.98 126.9999 0)
+    (property "Value" "1u" (id 1) (at 220.98 126.9999 0)
       (effects (font (size 1.27 1.27)) (justify left))
     )
@@
     )
     (property "Datasheet" "~" (id 3) (at 215.9 125.73 0)
+      (effects (font (size 1.27 1.27)) hide)
+    )
+    (pin "1")
+    (pin "2")
+  )
+  (symbol (lib_id "Device:R") (at 40.64 115.57 0) (unit 1)
+    (in_bom yes) (on_board yes) (fields_autoplaced)
+    (property "Reference" "R4" (id 0) (at 43.18 114.2999 0)
+      (effects (font (size 1.27 1.27)) (justify left))
+    )
+    (property "Value" "500k" (id 1) (at 43.18 116.8399 0)
+      (effects (font (size 1.27 1.27)) (justify left))
+    )
+    (property "Footprint" "Resistor_SMD:R_1206_3216Metric" (id 2) (at 38.862 115.57 90)
+      (effects (font (size 1.27 1.27)) hide)
+    )
+    (property "Datasheet" "~" (id 3) (at 40.64 115.57 0)
       (effects (font (size 1.27 1.27)) hide)
     )
@@
     (pin "1")
   )
-  (symbol (lib_id "Device:R") (at 49.53 121.92 0) (unit 1)
-    (in_bom yes) (on_board yes) (fields_autoplaced)
-    (property "Reference" "R4" (id 0) (at 52.07 120.6499 0)
-      (effects (font (size 1.27 1.27)) (justify left))
-    )
-    (property "Value" "1M" (id 1) (at 52.07 123.1899 0)
-      (effects (font (size 1.27 1.27)) (justify left))
-    )
-    (property "Footprint" "Resistor_SMD:R_1206_3216Metric" (id 2) (at 47.752 121.92 90)
-      (effects (font (size 1.27 1.27)) hide)
-    )
-    (property "Datasheet" "~" (id 3) (at 49.53 121.92 0)
-      (effects (font (size 1.27 1.27)) hide)
-    )
-    (pin "1")
-    (pin "2")
-  )
   (symbol (lib_id "Transistor_BJT:MMBT3904") (at 140.97 123.19 0) (unit 1)
     (in_bom yes) (on_board yes) (fields_autoplaced)
@@
     )
     (property "Datasheet" "~" (id 3) (at 231.14 106.68 0)
+      (effects (font (size 1.27 1.27)) hide)
+    )
+    (pin "1")
+    (pin "2")
+  )
+  (symbol (lib_id "Device:R") (at 40.64 107.95 0) (unit 1)
+    (in_bom yes) (on_board yes) (fields_autoplaced)
+    (property "Reference" "R3" (id 0) (at 43.18 106.6799 0)
+      (effects (font (size 1.27 1.27)) (justify left))
+    )
+    (property "Value" "500k" (id 1) (at 43.18 109.2199 0)
+      (effects (font (size 1.27 1.27)) (justify left))
+    )
+    (property "Footprint" "Resistor_SMD:R_1206_3216Metric" (id 2) (at 38.862 107.95 90)
+      (effects (font (size 1.27 1.27)) hide)
+    )
+    (property "Datasheet" "~" (id 3) (at 40.64 107.95 0)
       (effects (font (size 1.27 1.27)) hide)
     )
@@
     )
     (pin "1")
+  )
+  (symbol (lib_id "Device:R") (at 45.72 129.54 90) (unit 1)
+    (in_bom yes) (on_board yes)
+    (property "Reference" "R29" (id 0) (at 45.72 127 90))
+    (property "Value" "500k" (id 1) (at 45.72 132.08 90))
+    (property "Footprint" "Resistor_SMD:R_1206_3216Metric" (id 2) (at 45.72 131.318 90)
+      (effects (font (size 1.27 1.27)) hide)
+    )
+    (property "Datasheet" "~" (id 3) (at 45.72 129.54 0)
+      (effects (font (size 1.27 1.27)) hide)
+    )
+    (pin "1")
+    (pin "2")
   )
   (symbol (lib_id "VRB1205YMD-6WR3:VRB1205YMD-6WR3") (at 113.03 63.5 0) (mirror y) (unit 1)
@@
     )
     (pin "1")
-  )
-  (symbol (lib_id "Device:R") (at 49.53 113.03 0) (unit 1)
-    (in_bom yes) (on_board yes) (fields_autoplaced)
-    (property "Reference" "R3" (id 0) (at 52.07 111.7599 0)
-      (effects (font (size 1.27 1.27)) (justify left))
-    )
-    (property "Value" "1M" (id 1) (at 52.07 114.2999 0)
-      (effects (font (size 1.27 1.27)) (justify left))
-    )
-    (property "Footprint" "Resistor_SMD:R_1206_3216Metric" (id 2) (at 47.752 113.03 90)
-      (effects (font (size 1.27 1.27)) hide)
-    )
-    (property "Datasheet" "~" (id 3) (at 49.53 113.03 0)
-      (effects (font (size 1.27 1.27)) hide)
-    )
-    (pin "1")
-    (pin "2")
   )
   (symbol (lib_id "Device:LED") (at 152.4 147.32 90) (unit 1)
@@
     (pin "1")
   )
+  (symbol (lib_id "Device:R") (at 40.64 123.19 0) (unit 1)
+    (in_bom yes) (on_board yes) (fields_autoplaced)
+    (property "Reference" "R28" (id 0) (at 43.18 121.9199 0)
+      (effects (font (size 1.27 1.27)) (justify left))
+    )
+    (property "Value" "500k" (id 1) (at 43.18 124.4599 0)
+      (effects (font (size 1.27 1.27)) (justify left))
+    )
+    (property "Footprint" "Resistor_SMD:R_1206_3216Metric" (id 2) (at 38.862 123.19 90)
+      (effects (font (size 1.27 1.27)) hide)
+    )
+    (property "Datasheet" "~" (id 3) (at 40.64 123.19 0)
+      (effects (font (size 1.27 1.27)) hide)
+    )
+    (pin "1")
+    (pin "2")
+  )
   (symbol (lib_id "power_symbols:TS-") (at 88.9 106.68 0) (mirror y) (unit 1)
     (in_bom yes) (on_board yes)
@@
     )
     (path "/6419ca2c-ef5a-4147-ac00-395813048e0c"
-      (reference "C4") (unit 1) (value "1microF") (footprint "Capacitor_SMD:C_0603_1608Metric")
+      (reference "C4") (unit 1) (value "1u") (footprint "Capacitor_SMD:C_0603_1608Metric")
     )
     (path "/88ef39ab-6a5b-4e63-a663-ccc8204c87da"
@@
     )
     (path "/f2108bfb-38ea-4e94-955c-eefc1ef519d2/1cdd4cfa-6528-4292-a4d5-8830a935a03a"
-      (reference "C7") (unit 1) (value "0.1u") (footprint "Capacitor_SMD:C_0603_1608Metric")
+      (reference "C7") (unit 1) (value "100nF") (footprint "Capacitor_SMD:C_0603_1608Metric")
     )
     (path "/f2108bfb-38ea-4e94-955c-eefc1ef519d2/7ac41e2d-3759-481b-8346-cf965e811492"
@@
       (reference "R2") (unit 1) (value "2.2k") (footprint "Resistor_SMD:R_0603_1608Metric")
     )
-    (path "/a6228705-23bd-482f-acca-7da2e14116c4"
-      (reference "R3") (unit 1) (value "1M") (footprint "Resistor_SMD:R_1206_3216Metric")
-    )
-    (path "/777d367a-b25f-403a-ba4e-0f6fae2baddb"
-      (reference "R4") (unit 1) (value "1M") (footprint "Resistor_SMD:R_1206_3216Metric")
+    (path "/93996bd3-eaba-4d43-a446-a8ebba775afc"
+      (reference "R3") (unit 1) (value "500k") (footprint "Resistor_SMD:R_1206_3216Metric")
+    )
+    (path "/6eabfb58-c943-42b0-8750-8e0726977666"
+      (reference "R4") (unit 1) (value "500k") (footprint "Resistor_SMD:R_1206_3216Metric")
     )
     (path "/b46d17af-2d56-4e98-9e0f-528ad8a701eb"
@@
       (reference "R27") (unit 1) (value "500k") (footprint "Resistor_SMD:R_1206_3216Metric")
     )
+    (path "/ef308038-edc8-449c-b98b-6fa7c6dbe60b"
+      (reference "R28") (unit 1) (value "500k") (footprint "Resistor_SMD:R_1206_3216Metric")
+    )
+    (path "/a25087eb-7b6b-4391-9c39-fc1b08e772cd"
+      (reference "R29") (unit 1) (value "500k") (footprint "Resistor_SMD:R_1206_3216Metric")
+    )
     (path "/9e8d90fe-a30d-4bac-bfae-551e80945ffc"

Commit message: Fixed drc violations
Parts:
- added H1, H2, H3, H4: MountingHole, symbol Mechanical:MountingHole
Changed lines of the file:
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@@
     (pin "2")
+  )
+  (symbol (lib_id "Mechanical:MountingHole") (at 30.48 179.07 0) (unit 1)
+    (in_bom yes) (on_board yes)
+    (property "Reference" "H3" (id 0) (at 30.48 173.99 0))
+    (property "Value" "MountingHole" (id 1) (at 30.48 175.895 0))
+    (property "Footprint" "" (id 2) (at 30.48 179.07 0)
+      (effects (font (size 1.27 1.27)) hide)
+    )
+    (property "Datasheet" "~" (id 3) (at 30.48 179.07 0)
+      (effects (font (size 1.27 1.27)) hide)
+    )
   )
   (symbol (lib_id "power:+12V") (at 177.8 95.25 0) (unit 1)
@@
     (pin "1")
   )
+  (symbol (lib_id "Mechanical:MountingHole") (at 30.48 185.42 270) (unit 1)
+    (in_bom yes) (on_board yes) (fields_autoplaced)
+    (property "Reference" "H4" (id 0) (at 33.02 184.1499 90)
+      (effects (font (size 1.27 1.27)) (justify left))
+    )
+    (property "Value" "MountingHole" (id 1) (at 33.02 186.6899 90)
+      (effects (font (size 1.27 1.27)) (justify left))
+    )
+    (property "Footprint" "" (id 2) (at 30.48 185.42 0)
+      (effects (font (size 1.27 1.27)) hide)
+    )
+    (property "Datasheet" "~" (id 3) (at 30.48 185.42 0)
+      (effects (font (size 1.27 1.27)) hide)
+    )
+  )
   (symbol (lib_id "Device:LED") (at 152.4 147.32 90) (unit 1)
     (in_bom yes) (on_board yes) (fields_autoplaced)
@@
     (pin "1")
     (pin "2")
+  )
+  (symbol (lib_id "Mechanical:MountingHole") (at 30.48 170.18 0) (unit 1)
+    (in_bom yes) (on_board yes)
+    (property "Reference" "H2" (id 0) (at 30.48 165.1 0))
+    (property "Value" "MountingHole" (id 1) (at 30.48 167.005 0))
+    (property "Footprint" "" (id 2) (at 30.48 170.18 0)
+      (effects (font (size 1.27 1.27)) hide)
+    )
+    (property "Datasheet" "~" (id 3) (at 30.48 170.18 0)
+      (effects (font (size 1.27 1.27)) hide)
+    )
   )
   (symbol (lib_id "Device:R") (at 215.9 113.03 0) (unit 1)
@@
     (pin "1")
   )
+  (symbol (lib_id "Mechanical:MountingHole") (at 30.48 161.29 0) (unit 1)
+    (in_bom yes) (on_board yes)
+    (property "Reference" "H1" (id 0) (at 30.48 156.21 0))
+    (property "Value" "MountingHole" (id 1) (at 30.48 158.115 0))
+    (property "Footprint" "" (id 2) (at 30.48 161.29 0)
+      (effects (font (size 1.27 1.27)) hide)
+    )
+    (property "Datasheet" "~" (id 3) (at 30.48 161.29 0)
+      (effects (font (size 1.27 1.27)) hide)
+    )
+  )
   (symbol (lib_id "Device:R") (at 152.4 139.7 180) (unit 1)
     (in_bom yes) (on_board yes) (fields_autoplaced)
@@
       (reference "D12") (unit 1) (value "SMAJ15CA") (footprint "Diode_SMD:D_SMA")
     )
+    (path "/f123d011-8533-40fd-8ceb-1d6d6524727f"
+      (reference "H1") (unit 1) (value "MountingHole") (footprint "")
+    )
+    (path "/bafcf26a-004b-4146-93fd-c626c99f1dfd"
+      (reference "H2") (unit 1) (value "MountingHole") (footprint "")
+    )
+    (path "/46387f4a-380a-4037-8a88-083d0aa980c8"
+      (reference "H3") (unit 1) (value "MountingHole") (footprint "")
+    )
+    (path "/a83de003-e709-4dbc-90c8-09ed771dc320"
+      (reference "H4") (unit 1) (value "MountingHole") (footprint "")
+    )
     (path "/c7d8bc58-18ff-453c-8478-ea4fc1d31683"

Commit message: TSAL W/ updated DC-DC + Meme
Parts:
- removed U3: VRB1205YMD-6WR3, VRB1205YMD-6WR3:VRB1205YMD-6WR3, symbol VRB1205YMD-6WR3:VRB1205YMD-6WR3
- added U3: VRB1205YMD-15WR3, VRB1205YMD-6WR3:VRB1205YMD-15WR3, symbol VRB1205YMD-6WR3:VRB1205YMD-15WR3
Connections:
- net +12V: now also U3.1 (Ctrl), U3.3 (Vin)
- net +5V: now also U3.4 (+Vo)
- net GND: now also U3.2 (GND)
- net TS-: now also U3.6 (0V)
- no-connect marks 0 -> 1
Other:
- moved on the sheet: C1, C2, D4
