File: TSAL/PCB.kicad_sch (KiCad schematic)
At the start: 44 parts, among them J1 TE 770966-2, J2 JST B04B-XASK, Q1 IRLZ44N, Q2 MMBT3904, Q3 IRLZ44N, U1 TL431D, U2 LMV331, U3 VRB1205YMD-15WR3, U4 LTV-817S, U5 LM555xN

Commit message: New TSAL
Parts:
- removed C1, C2: 100u, Capacitor_SMD:CP_Elec_6.3x7.7, symbol Device:C_Polarized
- removed C3: 100nF, Capacitor_SMD:C_0603_1608Metric, symbol pspice:CAP
- removed C4: 1u, Capacitor_SMD:C_0603_1608Metric, symbol pspice:CAP
- removed D4: SMAJ15CA, Diode_SMD:D_SMA, symbol Device:D_TVS
- removed U3: VRB1205YMD-15WR3, VRB1205YMD-6WR3:VRB1205YMD-15WR3, symbol VRB1205YMD-6WR3:VRB1205YMD-15WR3
- added C1: 100n, symbol Device:C_Small
- added C10, C9: 500V 3.9u, symbol Device:C_Small
- added C11, C13: 10u, symbol Device:C_Small
- added C12, C14: 0.1u, symbol Device:C_Small
- added C2: 100u, symbol Device:C_Small
- added C3: 100n, symbol Device:C
- added C4: 1u, symbol Device:C
- added C7: C_Small, symbol Device:C_Small
- added D4: D_Schottky, symbol Device:D_Schottky
- added D6: D, symbol Device:D
- added D7: LED, symbol Device:LED
- added J3, J4: Conn_01x02, symbol Connector_Generic:Conn_01x02
- added L1: L, symbol Device:L
- added L2: 1m, symbol Device:L
- added R17, R18: 5k, symbol Device:R_Small
- added R19: 1k, symbol Device:R
- added R21: 0, symbol Device:R_Small
- added U3: UCC12040DVE, SO_0DVER_TEX, symbol 2023-11-19_21-51-37:UCC12040DVE
- added U7: MP174AGJ-Z, TSOT23-5_MP174A_MNP, symbol 2023-11-19_21-55-29:MP174AGJ-Z
- Q1, Q3: footprint Package_TO_SOT_SMD:TO-263-2 -> Package_TO_SOT_THT:TO-220-3_Vertical
- R15: value 2.2k -> 1k
- U5: footprint Package_SO:SOIC-8_3.9x4.9mm_P1.27mm -> Package_DIP:DIP-8_W7.62mm
Connections:
- net +12V: now also J2.1 (Pin_1); no longer C6.1, R11.1, R15.2, R9.2, U4.4, U5.8 (VCC)
- net +5V: now also C11.1, C12.1, C2.1, D6.2 (A), L1.2, U3.1 (EN), U3.3 (VINP)
- net GND: now also C13.2, C14.2, C3.1, C4.1, D7.1 (K), J3.2 (Pin_2), J4.2 (Pin_2), U3.10 (NC), U3.11 (NC), U3.12 (NC), U3.15 (GNDS), U3.16 (GNDS), U3.9 (GNDS); no longer J2.2 (Pin_2)
- net TS+: now also C10.1, L2.1
- net TS-: now also C10.2, C11.2, C12.2, C2.2, C9.2, D4.2 (A), U3.2 (GNDP), U3.4 (SYNC), U3.5 (SYNC_OK), U3.6 (NC), U3.7 (NC), U3.8 (NC)
- net at U5.5 (CV): now also C3.2
- net at R12.2, U5.2 (TR), U5.6 (THR): now also C4.2
- net at D5.2 (A): now also J4.1 (Pin_1); no longer J2.1 (Pin_1)
- new net: R21.1, U3.13 (SEL)
- new net: D7.2 (A), R19.1
- new net: C1.1, D6.1 (K), R17.1
- new net: R17.2, R18.1, U7.2 (FB)
- new net: C1.2, C7.2, D4.1 (K), L1.1, R18.2, U7.3 (SOURCE), U7.4 (SOURCE)
- new net: C9.1, L2.2, U7.5 (DRAIN)
- new net: C7.1, U7.1 (VCC)
- new net +5V@GLV: C13.1, C14.1, C6.1, J2.2 (Pin_2), J3.1 (Pin_1), R11.1, R15.2, R19.2, R21.2, R9.2, U3.14 (VISO), U4.4, U5.8 (VCC)
- no-connect marks 1 -> 0
Other:
- removed sheet Voltage Indicator
- note added: "Voltage Indicator"
- moved on the sheet: D5, J1

Commit message: TSAL V2
Parts:
- C1, C11, C12, C13, C14, C2, C3, C4: footprint (none) -> Capacitor_SMD:C_0603_1608Metric
- C10, C9: footprint (none) -> Capacitor_SMD:C_Elec_10x10.2
- C5, C6: value 100nF -> 100n
- C7: value C_Small -> 2.2u; footprint (none) -> Capacitor_SMD:C_0603_1608Metric
- D4: value D_Schottky -> AES2JF-HF; footprint (none) -> KiCADv6:CR_SMAF_CIP
- D6: value D -> 1N4007; footprint (none) -> Diode_SMD:D_SOD-123
- D7: value LED -> LED-Red; footprint (none) -> LED_SMD:LED_0603_1608Metric
- H1, H2, H3, H4: footprint (none) -> MountingHole:MountingHole_4mm
- J3, J4: footprint (none) -> Connector_TE-Connectivity:TE_MATE-N-LOK_1-770966-x_1x02_P4.14mm_Horizontal
- L1: value L -> 1.2m; footprint (none) -> Inductor_SMD:L_1008_2520Metric
- L2: footprint (none) -> Inductor_SMD:L_1008_2520Metric
- Q1, Q3: footprint Package_TO_SOT_THT:TO-220-3_Vertical -> IRLZ44NSTRLPBF:NMOSGDS_D2PAK_INF
- R17, R18, R19, R21: footprint (none) -> Resistor_SMD:R_0603_1608Metric
- U3: footprint SO_0DVER_TEX -> footprints:SO_0DVER_TEX
- U5: footprint Package_DIP:DIP-8_W7.62mm -> footprints 555:M08A-L
- U7: footprint TSOT23-5_MP174A_MNP -> MP174AGJ_Z:TSOT23-5_MP174A_MNP
